Commit message: fixing include related issues

File: urdf/barista.xacro (robot description, xacro)
@@ -2,6 +2,6 @@
 <robot name="BaristaII"
   xmlns:xacro="http://www.ros.org/wiki/xacro">
-  <xacro:include filename="$(find my_robot)/urdf/materials.xacro" />
-  <xacro:include filename="$(find my_robot)/urdf/barista.gazebo" />
+  <xacro:include filename="$(find barista_bot)/urdf/materials.xacro" />
+  <xacro:include filename="$(find barista_bot)/urdf/barista.gazebo" />
   <joint name="BaristaII__link_0_0_clone_JOINT_3" type="fixed">
     <parent link="left_rod"/>
@@ -255,5 +255,5 @@
       <origin rpy="0 0 0" xyz="0 0 0"/>
       <geometry>
-        <mesh filename="package://my_robot/meshes/hokuyo.dae" />
+        <mesh filename="package://barista_bot/meshes/hokuyo.dae" />
       </geometry>
     </visual>

Commit message: fixes

File: urdf/barista.xacro (robot description, xacro)
@@ -14,5 +14,5 @@
     <parent link="chassis"/>
     <child link="front_caster"/>
-    <origin rpy="0      -0.00014 -0.00024" xyz="0.19008 -0.04502 -0.00021"/>
+    <origin rpy="0      -0.00014 -0.00024" xyz="2.0004e-01  0 6.0000e-05"/>
     <axis xyz="0 0 0"/>
     <limit effort="0" lower="0" upper="0" velocity="0"/>
@@ -21,5 +21,5 @@
     <parent link="chassis"/>
     <child link="back_caster"/>
-    <origin rpy="0      -0.00029 -0.00049" xyz="-2.0004e-01  0.0000e-05 -6.0000e-05"/>
+    <origin rpy="0      -0.00029 -0.00049" xyz="-2.0004e-01  0 -6.0000e-05"/>
     <axis xyz="0 0 0"/>
     <limit effort="0" lower="0" upper="0" velocity="0"/>
@@ -97,11 +97,11 @@
       <origin rpy="0 0 0" xyz="0 0 0"/>
       <geometry>
-        <sphere radius="0.04"/>
-      </geometry>
-    </collision>
-    <visual>
-      <origin rpy="0 0 0" xyz="0 0 0"/>
-      <geometry>
-        <sphere radius="0.04"/>
+        <sphere radius="0.049"/>
+      </geometry>
+    </collision>
+    <visual>
+      <origin rpy="0 0 0" xyz="0 0 0"/>
+      <geometry>
+        <sphere radius="0.049"/>
       </geometry>
     </visual>
@@ -135,11 +135,11 @@
       <origin rpy="0 0 0" xyz="0 0 0"/>
       <geometry>
-        <sphere radius="0.04"/>
-      </geometry>
-    </collision>
-    <visual>
-      <origin rpy="0 0 0" xyz="0 0 0"/>
-      <geometry>
-        <sphere radius="0.04"/>
+        <sphere radius="0.049"/>
+      </geometry>
+    </collision>
+    <visual>
+      <origin rpy="0 0 0" xyz="0 0 0"/>
+      <geometry>
+        <sphere radius="0.049"/>
       </geometry>
     </visual>

File: urdf/my_robot.xacro (robot description, xacro)
@@ -14,5 +14,5 @@
     <material>Gazebo/Gray</material>
   </gazebo>
-  <xacro:include filename="$(find my_robot)/urdf/my_robot.gazebo" />
+  <xacro:include filename="$(find barista_bot)/urdf/my_robot.gazebo" />
   <link name="robot_footprint"></link>
   <joint name="robot_footprint_joint" type="fixed">
@@ -158,5 +158,5 @@
       <origin xyz="0  0  0" rpy=" 0  0  0"/>
       <geometry>
-        <mesh filename="package://my_robot/meshes/hokuyo.dae" />
+        <mesh filename="package://barista_bot/meshes/hokuyo.dae" />
       </geometry>
     </visual>

Commit message: update with macros

File: urdf/barista.xacro (robot description, xacro)
@@ -4,4 +4,9 @@
   <xacro:include filename="$(find barista_bot)/urdf/materials.xacro" />
   <xacro:include filename="$(find barista_bot)/urdf/barista.gazebo" />
+  <xacro:include filename="$(find barista_bot)/urdf/macros.xacro" />
+  <xacro:property name="casterRadius" value="0.049"/>
+  <xacro:property name="casterMass" value="1"/>
+  <xacro:property name="cameraSize" value="0.1"/>
+  <xacro:property name="cameraMass" value="0.5"/>
   <joint name="BaristaII__link_0_0_clone_JOINT_3" type="fixed">
     <parent link="left_rod"/>
@@ -71,123 +76,180 @@
   <link name="chassis">
     <inertial>
+      <mass value="5"/>
+      <origin rpy="0 0 0" xyz="0 0 0"/>
+      <inertia ixx="0.115625" ixy="0" ixz="0" iyy="0.115625" iyz="0" izz="0.15625"/>
+    </inertial>
+    <collision>
+      <origin rpy="0 0 0" xyz="0  0  0.2"/>
+      <geometry>
+        <cylinder length="0.3" radius="0.25"/>
+      </geometry>
+    </collision>
+    <visual>
+      <origin rpy="0 0 0" xyz="0  0  0.2"/>
+      <geometry>
+        <cylinder length="0.3" radius="0.25"/>
+      </geometry>
+    </visual>
+  </link>
+  <link name="front_caster">
+    <inertial>
+      <mass value="${casterMass}"/>
+      <origin rpy="0 0 0" xyz="0 0 0"/>
+      <sphere_inertia m="${casterMass}" r="${casterRadius}"/>
+    </inertial>
+    <collision>
+      <origin rpy="0 0 0" xyz="0 0 0"/>
+      <geometry>
+        <sphere radius="0.049"/>
+      </geometry>
+    </collision>
+    <visual>
+      <origin rpy="0 0 0" xyz="0 0 0"/>
+      <geometry>
+        <sphere radius="0.049"/>
+      </geometry>
+    </visual>
+  </link>
+  <link name="left_rod">
+    <inertial>
+      <mass value="0.5"/>
+      <origin rpy="0 0 0" xyz="0 0 0"/>
+      <inertia ixx="0.020467" ixy="0" ixz="0" iyy="0.020467" iyz="0" izz="0.0001"/>
+    </inertial>
+    <collision>
+      <origin rpy="0 0 0" xyz="0 0 0"/>
+      <geometry>
+        <cylinder length="0.7" radius="0.02"/>
+      </geometry>
+    </collision>
+    <visual>
+      <origin rpy="0 0 0" xyz="0 0 0"/>
+      <geometry>
+        <cylinder length="0.7" radius="0.02"/>
+      </geometry>
+    </visual>
+  </link>
+  <link name="back_caster">
+    <inertial>
+      <mass value="${casterMass}"/>
+      <origin rpy="0 0 0" xyz="0 0 0"/>
+      <sphere_inertia m="${casterMass}" r="${casterRadius}"/>
+    </inertial>
+    <collision>
+      <origin rpy="0 0 0" xyz="0 0 0"/>
+      <geometry>
+        <sphere radius="0.049"/>
+      </geometry>
+    </collision>
+    <visual>
+      <origin rpy="0 0 0" xyz="0 0 0"/>
+      <geometry>
+        <sphere radius="0.049"/>
+      </geometry>
+    </visual>
+  </link>
+  <link name="right_rod">
+    <inertial>
+      <mass value="0.5"/>
+      <origin rpy="0 0 0" xyz="0 0 0"/>
+      <inertia ixx="0.020467" ixy="0" ixz="0" iyy="0.020467" iyz="0" izz="0.0001"/>
+    </inertial>
+    <collision>
+      <origin rpy="0 0 0" xyz="0 0 0"/>
+      <geometry>
+        <cylinder length="0.7" radius="0.02"/>
+      </geometry>
+    </collision>
+    <visual>
+      <origin rpy="0 0 0" xyz="0 0 0"/>
+      <geometry>
+        <cylinder length="0.7" radius="0.02"/>
+      </geometry>
+    </visual>
+  </link>
+  <link name="top_plate">
+    <inertial>
+      <mass value="2"/>
+      <origin rpy="0 0 0" xyz="0 0 0"/>
+      <inertia ixx="0.032917" ixy="0" ixz="0" iyy="0.032917" iyz="0" izz="0.0625"/>
+    </inertial>
+    <collision>
+      <origin rpy="0 0 0" xyz="0 0 0"/>
+      <geometry>
+        <cylinder length="0.1" radius="0.25"/>
+      </geometry>
+    </collision>
+    <visual>
+      <origin rpy="0 0 0" xyz="0 0 0"/>
+      <geometry>
+        <cylinder length="0.1" radius="0.25"/>
+      </geometry>
+    </visual>
+  </link>
+  <link name="camera">
+    <inertial>
       <mass value="1"/>
       <origin rpy="0 0 0" xyz="0 0 0"/>
+      <inertia ixx="0.166667" ixy="0" ixz="0" iyy="0.166667" iyz="0" izz="0.166667"/>
+    </inertial>
+    <collision>
+      <origin rpy="0 0 0" xyz="0 0 0"/>
+      <geometry>
+        <box size="${cameraSize} ${cameraSize} ${cameraSize}"/>
+      </geometry>
+    </collision>
+    <visual>
+      <origin rpy="0 0 0" xyz="0 0 0"/>
+      <geometry>
+        <box size="${cameraSize} ${cameraSize} ${cameraSize}"/>
+      </geometry>
+    </visual>
+  </link>
+  <link name="left_wheel">
+    <inertial>
+      <mass value="${cameraMass}" />
+      <origin rpy=" 0  1.5707  1.5707" xyz="0 0 0"/>
+      <box_inertia m="${cameraMass}" x="${cameraSize}" y="${cameraSize}" z="${cameraSize}" />
+    </inertial>
+    <collision>
+      <origin rpy=" 0  1.5707  1.5707" xyz="0 0 0"/>
+      <geometry>
+        <cylinder length="0.1" radius="0.15"/>
+      </geometry>
+    </collision>
+    <visual>
+      <origin rpy=" 0  1.5707  1.5707" xyz="0 0 0"/>
+      <geometry>
+        <cylinder length="0.1" radius="0.15"/>
+      </geometry>
+    </visual>
+  </link>
+  <link name="right_wheel">
+    <inertial>
+      <mass value="1"/>
+      <origin rpy=" 0  1.5707  1.5707" xyz="0 0 0"/>
       <inertia ixx="0.145833" ixy="0" ixz="0" iyy="0.145833" iyz="0" izz="0.125"/>
     </inertial>
     <collision>
-      <origin rpy="0 0 0" xyz="0  0  0.2"/>
-      <geometry>
-        <cylinder length="0.3" radius="0.25"/>
-      </geometry>
-    </collision>
-    <visual>
-      <origin rpy="0 0 0" xyz="0  0  0.2"/>
-      <geometry>
-        <cylinder length="0.3" radius="0.25"/>
-      </geometry>
-    </visual>
-  </link>
-  <link name="front_caster">
+      <origin rpy=" 0  1.5707  1.5707" xyz="0 0 0"/>
+      <geometry>
+        <cylinder length="0.1" radius="0.15"/>
+      </geometry>
+    </collision>
+    <visual>
+      <origin rpy=" 0  1.5707  1.5707" xyz="0 0 0"/>
+      <geometry>
+        <cylinder length="0.1" radius="0.15"/>
+      </geometry>
+    </visual>
+  </link>
+  <link name="hokuyo">
     <inertial>
       <mass value="1"/>
       <origin rpy="0 0 0" xyz="0 0 0"/>
-      <inertia ixx="0.1" ixy="0" ixz="0" iyy="0.1" iyz="0" izz="0.1"/>
-    </inertial>
-    <collision>
-      <origin rpy="0 0 0" xyz="0 0 0"/>
-      <geometry>
-        <sphere radius="0.049"/>
-      </geometry>
-    </collision>
-    <visual>
-      <origin rpy="0 0 0" xyz="0 0 0"/>
-      <geometry>
-        <sphere radius="0.049"/>
-      </geometry>
-    </visual>
-  </link>
-  <link name="left_rod">
-    <inertial>
-      <mass value="1"/>
-      <origin rpy="0 0 0" xyz="0 0 0"/>
-      <inertia ixx="0.145833" ixy="0" ixz="0" iyy="0.145833" iyz="0" izz="0.125"/>
-    </inertial>
-    <collision>
-      <origin rpy="0 0 0" xyz="0 0 0"/>
-      <geometry>
-        <cylinder length="0.7" radius="0.02"/>
-      </geometry>
-    </collision>
-    <visual>
-      <origin rpy="0 0 0" xyz="0 0 0"/>
-      <geometry>
-        <cylinder length="0.7" radius="0.02"/>
-      </geometry>
-    </visual>
-  </link>
-  <link name="back_caster">
-    <inertial>
-      <mass value="1"/>
-      <origin rpy="0 0 0" xyz="0 0 0"/>
-      <inertia ixx="0.1" ixy="0" ixz="0" iyy="0.1" iyz="0" izz="0.1"/>
-    </inertial>
-    <collision>
-      <origin rpy="0 0 0" xyz="0 0 0"/>
-      <geometry>
-        <sphere radius="0.049"/>
-      </geometry>
-    </collision>
-    <visual>
-      <origin rpy="0 0 0" xyz="0 0 0"/>
-      <geometry>
-        <sphere radius="0.049"/>
-      </geometry>
-    </visual>
-  </link>
-  <link name="right_rod">
-    <inertial>
-      <mass value="1"/>
-      <origin rpy="0 0 0" xyz="0 0 0"/>
-      <inertia ixx="0.145833" ixy="0" ixz="0" iyy="0.145833" iyz="0" izz="0.125"/>
-    </inertial>
-    <collision>
-      <origin rpy="0 0 0" xyz="0 0 0"/>
-      <geometry>
-        <cylinder length="0.7" radius="0.02"/>
-      </geometry>
-    </collision>
-    <visual>
-      <origin rpy="0 0 0" xyz="0 0 0"/>
-      <geometry>
-        <cylinder length="0.7" radius="0.02"/>
-      </geometry>
-    </visual>
-  </link>
-  <link name="top_plate">
-    <inertial>
-      <mass value="1"/>
-      <origin rpy="0 0 0" xyz="0 0 0"/>
-      <inertia ixx="0.145833" ixy="0" ixz="0" iyy="0.145833" iyz="0" izz="0.125"/>
-    </inertial>
-    <collision>
-      <origin rpy="0 0 0" xyz="0 0 0"/>
-      <geometry>
-        <cylinder length="0.1" radius="0.25"/>
-      </geometry>
-    </collision>
-    <visual>
-      <origin rpy="0 0 0" xyz="0 0 0"/>
-      <geometry>
-        <cylinder length="0.1" radius="0.25"/>
-      </geometry>
-    </visual>
-  </link>
-  <link name="camera">
-    <inertial>
-      <mass value="1"/>
-      <origin rpy="0 0 0" xyz="0 0 0"/>
       <inertia ixx="0.166667" ixy="0" ixz="0" iyy="0.166667" iyz="0" izz="0.166667"/>
     </inertial>
-    <collision>
+    <collision name="BaristaII__collision">
       <origin rpy="0 0 0" xyz="0 0 0"/>
       <geometry>
@@ -195,61 +257,4 @@
       </geometry>
     </collision>
-    <visual>
-      <origin rpy="0 0 0" xyz="0 0 0"/>
-      <geometry>
-        <box size="0.1 0.1 0.1"/>
-      </geometry>
-    </visual>
-  </link>
-  <link name="left_wheel">
-    <inertial>
-      <mass value="1"/>
-      <origin rpy=" 0  1.5707  1.5707" xyz="0 0 0"/>
-      <inertia ixx="0.145833" ixy="0" ixz="0" iyy="0.145833" iyz="0" izz="0.125"/>
-    </inertial>
-    <collision>
-      <origin rpy=" 0  1.5707  1.5707" xyz="0 0 0"/>
-      <geometry>
-        <cylinder length="0.1" radius="0.15"/>
-      </geometry>
-    </collision>
-    <visual>
-      <origin rpy=" 0  1.5707  1.5707" xyz="0 0 0"/>
-      <geometry>
-        <cylinder length="0.1" radius="0.15"/>
-      </geometry>
-    </visual>
-  </link>
-  <link name="right_wheel">
-    <inertial>
-      <mass value="1"/>
-      <origin rpy=" 0  1.5707  1.5707" xyz="0 0 0"/>
-      <inertia ixx="0.145833" ixy="0" ixz="0" iyy="0.145833" iyz="0" izz="0.125"/>
-    </inertial>
-    <collision>
-      <origin rpy=" 0  1.5707  1.5707" xyz="0 0 0"/>
-      <geometry>
-        <cylinder length="0.1" radius="0.15"/>
-      </geometry>
-    </collision>
-    <visual>
-      <origin rpy=" 0  1.5707  1.5707" xyz="0 0 0"/>
-      <geometry>
-        <cylinder length="0.1" radius="0.15"/>
-      </geometry>
-    </visual>
-  </link>
-  <link name="hokuyo">
-    <inertial>
-      <mass value="1"/>
-      <origin rpy="0 0 0" xyz="0 0 0"/>
-      <inertia ixx="0.166667" ixy="0" ixz="0" iyy="0.166667" iyz="0" izz="0.166667"/>
-    </inertial>
-    <collision name="BaristaII__collision">
-      <origin rpy="0 0 0" xyz="0 0 0"/>
-      <geometry>
-        <box size="0.1 0.1 0.1"/>
-      </geometry>
-    </collision>
     <visual name="BaristaII__visual">
       <origin rpy="0 0 0" xyz="0 0 0"/>

Commit message: updating for amcl

File: urdf/barista.xacro (robot description, xacro)
@@ -9,4 +9,9 @@
   <xacro:property name="cameraSize" value="0.1"/>
   <xacro:property name="cameraMass" value="0.5"/>
+  <!-- <link name="base_link" />
+  <joint name="base_link_to_chassis" type="fixed">
+    <parent link="base_link"/>
+    <child link="chassis"/>
+  </joint> -->
   <joint name="BaristaII__link_0_0_clone_JOINT_3" type="fixed">
     <parent link="left_rod"/>
@@ -33,5 +38,5 @@
     <parent link="chassis"/>
     <child link="left_rod"/>
-    <origin rpy="0 0 0" xyz="0   -0.23  0.7"/>
+    <origin rpy="0 0 0" xyz="0   -0.23  0.5"/>
     <axis xyz="0 0 0"/>
     <limit effort="0" lower="0" upper="0" velocity="0"/>
@@ -40,5 +45,5 @@
     <parent link="chassis"/>
     <child link="right_rod"/>
-    <origin rpy="0 0 0" xyz="0      0.22999 0.7"/>
+    <origin rpy="0 0 0" xyz="0      0.22999 0.5"/>
     <axis xyz="0 0 0"/>
     <limit effort="0" lower="0" upper="0" velocity="0"/>
@@ -121,11 +126,11 @@
       <origin rpy="0 0 0" xyz="0 0 0"/>
       <geometry>
-        <cylinder length="0.7" radius="0.02"/>
-      </geometry>
-    </collision>
-    <visual>
-      <origin rpy="0 0 0" xyz="0 0 0"/>
-      <geometry>
-        <cylinder length="0.7" radius="0.02"/>
+        <cylinder length="0.3" radius="0.02"/>
+      </geometry>
+    </collision>
+    <visual>
+      <origin rpy="0 0 0" xyz="0 0 0"/>
+      <geometry>
+        <cylinder length="0.5" radius="0.02"/>
       </geometry>
     </visual>
@@ -159,11 +164,11 @@
       <origin rpy="0 0 0" xyz="0 0 0"/>
       <geometry>
-        <cylinder length="0.7" radius="0.02"/>
-      </geometry>
-    </collision>
-    <visual>
-      <origin rpy="0 0 0" xyz="0 0 0"/>
-      <geometry>
-        <cylinder length="0.7" radius="0.02"/>
+        <cylinder length="0.5" radius="0.02"/>
+      </geometry>
+    </collision>
+    <visual>
+      <origin rpy="0 0 0" xyz="0 0 0"/>
+      <geometry>
+        <cylinder length="0.5" radius="0.02"/>
       </geometry>
     </visual>
@@ -190,65 +195,65 @@
   <link name="camera">
     <inertial>
+      <mass value="0.1"/>
+      <origin rpy="0 0 0" xyz="0 0 0"/>
+      <inertia ixx="0.166667" ixy="0" ixz="0" iyy="0.166667" iyz="0" izz="0.166667"/>
+    </inertial>
+    <collision>
+      <origin rpy="0 0 0" xyz="0 0 0"/>
+      <geometry>
+        <box size="${cameraSize} ${cameraSize} ${cameraSize}"/>
+      </geometry>
+    </collision>
+    <visual>
+      <origin rpy="0 0 0" xyz="0 0 0"/>
+      <geometry>
+        <box size="${cameraSize} ${cameraSize} ${cameraSize}"/>
+      </geometry>
+    </visual>
+  </link>
+  <link name="left_wheel">
+    <inertial>
+      <mass value="${cameraMass}" />
+      <origin rpy=" 0  1.5707  1.5707" xyz="0 0 0"/>
+      <box_inertia m="${cameraMass}" x="${cameraSize}" y="${cameraSize}" z="${cameraSize}" />
+    </inertial>
+    <collision>
+      <origin rpy=" 0  1.5707  1.5707" xyz="0 0 0"/>
+      <geometry>
+        <cylinder length="0.1" radius="0.15"/>
+      </geometry>
+    </collision>
+    <visual>
+      <origin rpy=" 0  1.5707  1.5707" xyz="0 0 0"/>
+      <geometry>
+        <cylinder length="0.1" radius="0.15"/>
+      </geometry>
+    </visual>
+  </link>
+  <link name="right_wheel">
+    <inertial>
       <mass value="1"/>
+      <origin rpy=" 0  1.5707  1.5707" xyz="0 0 0"/>
+      <inertia ixx="0.145833" ixy="0" ixz="0" iyy="0.145833" iyz="0" izz="0.125"/>
+    </inertial>
+    <collision>
+      <origin rpy=" 0  1.5707  1.5707" xyz="0 0 0"/>
+      <geometry>
+        <cylinder length="0.1" radius="0.15"/>
+      </geometry>
+    </collision>
+    <visual>
+      <origin rpy=" 0  1.5707  1.5707" xyz="0 0 0"/>
+      <geometry>
+        <cylinder length="0.1" radius="0.15"/>
+      </geometry>
+    </visual>
+  </link>
+  <link name="hokuyo">
+    <inertial>
+      <mass value="0.1"/>
       <origin rpy="0 0 0" xyz="0 0 0"/>
       <inertia ixx="0.166667" ixy="0" ixz="0" iyy="0.166667" iyz="0" izz="0.166667"/>
     </inertial>
-    <collision>
-      <origin rpy="0 0 0" xyz="0 0 0"/>
-      <geometry>
-        <box size="${cameraSize} ${cameraSize} ${cameraSize}"/>
-      </geometry>
-    </collision>
-    <visual>
-      <origin rpy="0 0 0" xyz="0 0 0"/>
-      <geometry>
-        <box size="${cameraSize} ${cameraSize} ${cameraSize}"/>
-      </geometry>
-    </visual>
-  </link>
-  <link name="left_wheel">
-    <inertial>
-      <mass value="${cameraMass}" />
-      <origin rpy=" 0  1.5707  1.5707" xyz="0 0 0"/>
-      <box_inertia m="${cameraMass}" x="${cameraSize}" y="${cameraSize}" z="${cameraSize}" />
-    </inertial>
-    <collision>
-      <origin rpy=" 0  1.5707  1.5707" xyz="0 0 0"/>
-      <geometry>
-        <cylinder length="0.1" radius="0.15"/>
-      </geometry>
-    </collision>
-    <visual>
-      <origin rpy=" 0  1.5707  1.5707" xyz="0 0 0"/>
-      <geometry>
-        <cylinder length="0.1" radius="0.15"/>
-      </geometry>
-    </visual>
-  </link>
-  <link name="right_wheel">
-    <inertial>
-      <mass value="1"/>
-      <origin rpy=" 0  1.5707  1.5707" xyz="0 0 0"/>
-      <inertia ixx="0.145833" ixy="0" ixz="0" iyy="0.145833" iyz="0" izz="0.125"/>
-    </inertial>
-    <collision>
-      <origin rpy=" 0  1.5707  1.5707" xyz="0 0 0"/>
-      <geometry>
-        <cylinder length="0.1" radius="0.15"/>
-      </geometry>
-    </collision>
-    <visual>
-      <origin rpy=" 0  1.5707  1.5707" xyz="0 0 0"/>
-      <geometry>
-        <cylinder length="0.1" radius="0.15"/>
-      </geometry>
-    </visual>
-  </link>
-  <link name="hokuyo">
-    <inertial>
-      <mass value="1"/>
-      <origin rpy="0 0 0" xyz="0 0 0"/>
-      <inertia ixx="0.166667" ixy="0" ixz="0" iyy="0.166667" iyz="0" izz="0.166667"/>
-    </inertial>
     <collision name="BaristaII__collision">
       <origin rpy="0 0 0" xyz="0 0 0"/>

Commit message: adding RTAB mapping

File: urdf/barista.xacro (robot description, xacro)
@@ -269,3 +269,10 @@
     </visual>
   </link>
+  <joint name="camera_optical_joint" type="fixed">
+    <origin xyz="0 0 0" rpy="-1.5707 0 -1.5707"/>
+    <parent link="camera"/>
+    <child link="camera_link_optical"/>
+  </joint>
+  <link name="camera_link_optical">
+  </link>
 </robot>
